File: EsquematicoTaller2/EsquematicoTaller2.kicad_sch (KiCad schematic)
At the start: 5 parts, among them J1 Raspberry_Pi_2_3, J3 OV2640_Module, M1 Motor_Servo, SW1 Pulsador

Commit message: ultima actu
Connections:
- net PWM_SW: now also J1.10 (GPIO15/RXD); no longer J1.8 (GPIO14/TXD)
- net D0: now reaches J1.11 (GPIO17)
- net D0: now also J3.8 (D0)
- net DCLK: now reaches J1.12 (GPIO18/PWM0)
- net DCLK: now also J3.16 (DCLK)
- net D2: now reaches J1.13 (GPIO27)
- net D2: now also J3.10 (D2)
- net D3: now reaches J1.15 (GPIO22)
- net D3: now also J3.11 (D3)
- net at SW1.3 (B), SW1.4 (B): now also J1.33 (PWM1/GPIO13); no longer J1.16 (GPIO23)
- net D4: now reaches J1.18 (GPIO24)
- net D4: now also J3.12 (D4)
- net D6: now reaches J1.22 (GPIO25)
- net D6: now also J3.14 (D6)
- net D7: now reaches J1.29 (GCLK1/GPIO5)
- net D7: now also J3.15 (D7)
- net SDA: now reaches J1.3 (SDA/GPIO2)
- net SDA: now also J3.6 (SDA)
- net VSYNC: now reaches J1.35 (GPIO19/MISO1)
- net VSYNC: now also J3.3 (VSYNC)
- net RST: now reaches J1.37 (GPIO26)
- net RST: now also J3.7 (RST)
- net HREF: now reaches J1.38 (GPIO20/MOSI1)
- net HREF: now also J3.5 (HREF)
- net PWDN: now reaches J1.40 (GPIO21/SCLK1)
- net PWDN: now also J3.18 (PWDN)
- net SCL: now reaches J1.5 (SCL/GPIO3)
- net SCL: now also J3.4 (SCL)
- net D5: now reaches J3.13 (D5)
- net D5: now also J1.16 (GPIO23)
- net D1: now reaches J3.9 (D1)
- net D1: now also J1.8 (GPIO14/TXD)
Other:
- title: (none) -> A3B. FaceId de apple | Ring de amazon | nest de google
